File: hardware/kicad/DSR-1/DSR-1.kicad_sch (KiCad schematic)
At the start: 23 parts, among them Q2 MMBT3904, U10 STM32G0C1KCUx

Commit message: updated schematics
Parts:
- added C17, C21, C23, C25: 10uf, symbol Device:C_US
- added C18: 100nf, symbol Device:C_US
- added C19: 4.7uf, symbol Device:C_US
- added C20: 22uf, symbol Device:C_US
- added C22: 47uF 16V, symbol Device:C_US
- added C24, C26: 1uF, symbol Device:C_US
- added D12: USBLC6-2SC6Y, USBLC6-2SC6Y:SOT95P280X145-6N, symbol DSR-1:USBLC6-2SC6Y
- added D13, D14, D15, D16, D18: SS14, Diode_SMD:D_SMA, symbol Diode:SS14
- added D17: SMBJ12A-13-F, SMBJ12A-13-F:DIOM5336X250N, symbol SMBJ12A-13-F:SMBJ12A-13-F
- added F2: Polyfuse, symbol Device:Polyfuse
- added J3: USB_C_Receptacle, symbol DSR-1:USB_C_Receptacle
- added J4: Barrel_Jack, symbol Connector:Barrel_Jack
- added L3: 4.7uH 1.5A, symbol Device:L
- added L4: 4.7uH, symbol Device:L
- added R16: 100k, symbol Device:R
- added R17: 649k, symbol Device:R
- added R18: 169k, symbol Device:R
- added R19: 10k, symbol Device:R
- added U6: AP63203WU-7, AP63203WU-7:SOIC_05WU-7_DIO-M, symbol AP63203WU-7:AP63203WU-7
- added U7: IP2721, IP2721:TSSOP16, symbol DSR-1:IP2721
- added U8: MT3608, Package_TO_SOT_SMD:SOT-23-6, symbol DSR-1:MT3608
- added U9: MCP1700x-330xxTT, Package_TO_SOT_SMD:SOT-23, symbol DSR-1:MCP1700x-330xxTT
Connections:
- net +3.3V: now also C25.1, D12.5 (VBUS), U9.2 (VO)
- net B+1: now also C20.1, C21.1, C23.1, L3.2, R16.1, R17.1, R18.1, U8.4 (EN), U8.5 (IN), U9.3 (VI)
- net B+3: now also C22.1, D18.2 (A)
- net CC1: now also J3.A5 (CC1), U7.P$13 (CC1)
- net CC2: now also J3.B5 (CC2), U7.P$12 (CC2)
- net GND: now also C17.1, C17.2, C19.1, C19.2, C20.2, C21.2, C22.2, C24.2, C26.2, D12.2 (GND), D14.2 (A), D16.2 (A), D17.1, D17.2, F2.2, J3.A1 (GND), J3.A12 (GND), J3.B1 (GND), J3.B12 (GND), J3.SH (SHIELD), R16.2, R19.2, U6.2 (EN), U6.3 (VIN), U6.4 (GND), U7.P$11 (SEL), U7.P$16 (VBUS), U7.P$5 (GND), U8.2 (GND), U9.1 (GND)
- net USB_DM: now also D12.6 (I/O1_2)
- net USB_DP: now also D12.4 (I/O2_2)
- new net: D13.2 (A), D14.1 (K), J4.2
- new net: C18.1, U6.6 (BST)
- new net: C18.2, L3.1, U6.5 (SW)
- new net: D13.1 (K), D15.1 (K), F2.1
- new net: D18.1 (K), L4.2
- new net: R17.2, U6.1 (FB)
- new net: D15.2 (A), D16.1 (K), J4.1
- new net: L4.1, U8.1 (SW)
- new net: R18.2, R19.1, U8.3 (FB)
- new net: C25.2, C26.1
- new net: C23.2, C24.1
- new net: J3.A4 (VBUS), J3.A9 (VBUS), J3.B4 (VBUS), J3.B9 (VBUS), U7.P$1 (VBUSG), U7.P$2 (VIN)
- new net: D12.3 (I/O2_1), J3.A6 (D+), J3.B6 (D+)
- new net: D12.1 (I/O1_1), J3.A7 (D-), J3.B7 (D-)
Other:
- note added: "+"
- note added: "10v"
- note added: "16v"
- note added: "B+1 output = 0.8 × (1 + 649k/100k) = 6.19V EN tied to VIN - AP63203 internal clamp handles 9V input safely. C3 (BST cap) must be placed within 1mm of BST/SW pins on PCB."
- note added: "B+3 output = 0.6 × (1 + 169k/10k) = 10.74V nominal. ⚠ SW NODE: high dV/dt at 1.2MHz. Keep SW trace <3mm. Minimum 2mm clearance to FG, ADC, and motor drive signal traces. C8 must be 47µF (not 22µF) - X5R derating at 10.8V reduces effective capacitance. Use 16V rated part for adequate margin."
- note added: "BRING-UP ORDER: 1. Verify 9V_PD present before AP63203 powers up 2. Check B+1 = 6.0-6.2V before enabling downstream 3. Check B+3 = 10.5-11V (no load) 4. Check +3.3V = 3.3V ±2% 5. Do not connect WM-D6C harness until all rails verified"
- note added: "Fixed 3.3V LDO. VIN max 16V - B+1 = 6V nominal, margin adequate. Requires minimum 1µF on VOUT for stability - C7+C10 exceed this."
- note added: "SEL pin sets PD voltage request - verify correct resistor value against IP2721 datasheet for 9V profile before ordering PCB. VBUSG must be tied to VIN. Floating VBUSG prevents output enable after negotiation regardless of CC state."
- note added: "Variant A - USB-C PD/Data"
- note added: "Variant B - Barrel Jack, Polarity Agnostic"
- note added: "Variant B input: 9V DC nominal, 5.5mm/2.1mm barrel jack. Polarity agnostic - bridge rectifier output is always positive. Do NOT connect a 6V adapter - minimum 7.5V required after 0.8V bridge drop to maintain regulation headroom. SMBJ12A: standoff 12V, clamp 19.9V max. AP63203 VIN abs max 32V."
- moved on the sheet: C27, C28, C29, C30, C31, C32, D19, D20, D21, D22, Q2, R20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

Commit message: updated schematic guide and dsr-1 schematic
Parts:
- removed C17, C21, C23, C25: 10uf, symbol Device:C_US
- removed C18: 100nf, symbol Device:C_US
- removed C19: 4.7uf, symbol Device:C_US
- removed C20: 22uf, symbol Device:C_US
- removed C22: 47uF 16V, symbol Device:C_US
- removed C24, C26: 1uF, symbol Device:C_US
- removed D12: USBLC6-2SC6Y, USBLC6-2SC6Y:SOT95P280X145-6N, symbol DSR-1:USBLC6-2SC6Y
- removed D13, D14, D15, D16, D18: SS14, Diode_SMD:D_SMA, symbol Diode:SS14
- removed D17: SMBJ12A-13-F, SMBJ12A-13-F:DIOM5336X250N, symbol SMBJ12A-13-F:SMBJ12A-13-F
- removed F2: Polyfuse, symbol Device:Polyfuse
- removed J3: USB_C_Receptacle, symbol DSR-1:USB_C_Receptacle
- removed J4: Barrel_Jack, symbol Connector:Barrel_Jack
- removed L3: 4.7uH 1.5A, symbol Device:L
- removed L4: 4.7uH, symbol Device:L
- removed R16: 100k, symbol Device:R
- removed R17: 649k, symbol Device:R
- removed R18: 169k, symbol Device:R
- removed R19: 10k, symbol Device:R
- removed U6: AP63203WU-7, AP63203WU-7:SOIC_05WU-7_DIO-M, symbol AP63203WU-7:AP63203WU-7
- removed U7: IP2721, IP2721:TSSOP16, symbol DSR-1:IP2721
- removed U8: MT3608, Package_TO_SOT_SMD:SOT-23-6, symbol DSR-1:MT3608
- removed U9: MCP1700x-330xxTT, Package_TO_SOT_SMD:SOT-23, symbol DSR-1:MCP1700x-330xxTT
Other:
- note removed: "+"
- note removed: "10v"
- note removed: "16v"
- note removed: "B+1 output = 0.8 × (1 + 649k/100k) = 6.19V EN tied to VIN - AP63203 internal clamp handles 9V input safely. C3 (BST cap) must be placed within 1mm of BST/SW pins on PCB."
- note removed: "B+3 output = 0.6 × (1 + 169k/10k) = 10.74V nominal. ⚠ SW NODE: high dV/dt at 1.2MHz. Keep SW trace <3mm. Minimum 2mm clearance to FG, ADC, and motor drive signal traces. C8 must be 47µF (not 22µF) - X5R derating at 10.8V reduces effective capacitance. Use 16V rated part for adequate margin."
- note removed: "BRING-UP ORDER: 1. Verify 9V_PD present before AP63203 powers up 2. Check B+1 = 6.0-6.2V before enabling downstream 3. Check B+3 = 10.5-11V (no load) 4. Check +3.3V = 3.3V ±2% 5. Do not connect WM-D6C harness until all rails verified"
- note removed: "Fixed 3.3V LDO. VIN max 16V - B+1 = 6V nominal, margin adequate. Requires minimum 1µF on VOUT for stability - C7+C10 exceed this."
- note removed: "SEL pin sets PD voltage request - verify correct resistor value against IP2721 datasheet for 9V profile before ordering PCB. VBUSG must be tied to VIN. Floating VBUSG prevents output enable after negotiation regardless of CC state."
- note removed: "Variant A - USB-C PD/Data"
- note removed: "Variant B - Barrel Jack, Polarity Agnostic"
- note removed: "Variant B input: 9V DC nominal, 5.5mm/2.1mm barrel jack. Polarity agnostic - bridge rectifier output is always positive. Do NOT connect a 6V adapter - minimum 7.5V required after 0.8V bridge drop to maintain regulation headroom. SMBJ12A: standoff 12V, clamp 19.9V max. AP63203 VIN abs max 32V."
- moved on the sheet: C27, C28, C29, C30, C31, C32, D19, D20, D21, D22, Q2, R20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
