File: hardware/kicad/DSR-1/Power input zone.kicad_sch (KiCad schematic)
At the start: 0 parts

Commit message: Updated schematics
Changed lines of the file:
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@@
 	(generator_version "10.0")
 	(paper "A4")
+	(hierarchical_label "USB_DM"
+		(shape bidirectional)
+		(at 257.81 33.02 0)
+		(effects
+			(font
+				(size 1.27 1.27)
+			)
+			(justify left)
+		)
+	)
+	(hierarchical_label "CC2"
+		(shape bidirectional)
+		(at 260.35 44.45 0)
+		(effects
+			(font
+				(size 1.27 1.27)
+			)
+			(justify left)
+		)
+	)
+	(hierarchical_label "USB_DP"
+		(shape bidirectional)
+		(at 256.54 26.67 0)
+		(effects
+			(font
+				(size 1.27 1.27)
+			)
+			(justify left)
+		)
+	)
 	(hierarchical_label "9V_PD"
 		(shape output)
 		(at 31.75 36.83 0)
+		(effects
+			(font
+				(size 1.27 1.27)
+			)
+			(justify left)
+		)
+	)
+	(hierarchical_label "CC1"
+		(shape bidirectional)
+		(at 260.35 38.1 0)
 		(effects
 			(font
@@
 		(property "Reference" "#PWR03"
 			(at 121.9726 16.51 0)
-			(show_name no)
-			(do_not_autoplace no)
-			(effects
-				(font
-					(size 1.27 1.27)
-				)
-			)
-		)
-		(property "Value" ""
+			(hide yes)
+			(show_name no)
+			(do_not_autoplace no)
+			(effects
+				(font
+					(size 1.27 1.27)
+				)
+			)
+		)
+		(property "Value" "B+1"
 			(at 119.38 25.4 0)
+			(hide yes)
 			(show_name no)
 			(do_not_autoplace no)
@@
 		(property "Reference" "#PWR04"
 			(at 147.3726 15.24 0)
+			(hide yes)
 			(show_name no)
 			(do_not_autoplace no)
@@
 		(property "Value" "B+3"
 			(at 147.3726 17.78 0)
-			(show_name no)
-			(do_not_autoplace no)
+			(hide yes)
+			(show_name no)
+			(do_not_autoplace no)
