File: hardware/kicad/DSR-1/Power management.kicad_sch (KiCad schematic)
At the start: 0 parts

Commit message: Updated schematics
Changed lines of the file:
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@@
 	(generator_version "10.0")
 	(paper "A4")
-	(hierarchical_label "+3V3"
-		(shape output)
-		(at 255.27 24.13 0)
-		(effects
-			(font
-				(size 1.27 1.27)
-			)
-			(justify left)
-		)
-	)
 	(hierarchical_label "9V_PD"
 		(shape input)
@@
 		(effects
 			(font
-				(size 1.27 1.27)
-			)
-			(justify left)
-		)
-	)
-	(hierarchical_label "B+1"
-		(shape output)
-		(at 256.54 30.48 0)
-		(effects
-			(font
