File: hardware/kicad/DSR-1/STM32G0B1 and decoupling.kicad_sch (KiCad schematic)
At the start: 0 parts

Commit message: Updated schematics
Changed lines of the file:
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@@
 	(generator_version "10.0")
 	(paper "A4")
-	(hierarchical_label "MOTOR_DAC_OUT"
-		(shape output)
-		(at 245.11 20.32 0)
-		(effects
-			(font
-				(size 1.27 1.27)
-			)
-			(justify left)
-		)
-	)
 	(hierarchical_label "RV603_WIPER"
 		(shape input)
@@
 		(shape input)
 		(at 29.21 59.69 0)
-		(effects
-			(font
-				(size 1.27 1.27)
-			)
-			(justify left)
-		)
-	)
-	(hierarchical_label "+3V3"
-		(shape input)
-		(at 29.21 24.13 0)
 		(effects
 			(font
@@
 		(effects
 			(font
+				(size 1.27 1.27)
+			)
+			(justify left)
+		)
+	)
+	(hierarchical_label "SPEED_TUNE_SW"
+		(shape input)
+		(at 245.11 31.75 0)
+		(effects
+			(font
