File: hardware/kicad/DSR-1/STM32G0C1 and decoupling.kicad_sch (KiCad schematic)
At the start: 6 parts, among them U5 STM32G0C1KCUx

Commit message: completed schematics through sheet 5.
Changed lines of the file:
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@@
-		)
-	)
-	(label "DEBUG_TX"
-		(at 91.44 104.14 180)
-		(effects
-			(font
-				(size 1.27 1.27)
-			)
-			(justify right bottom)
 		)
 	)
@@
 		)
 	)
+	(hierarchical_label "DEBUG_TX"
+		(shape input)
+		(at 91.44 104.14 180)
+		(effects
+			(font
+				(size 1.27 1.27)
+			)
+			(justify right)
+		)
+	)
